File: KiCad/picoswitch.kicad_pcb (KiCad board)
At the start: 2 copper layers, 41.5 x 66 mm, 7 parts, among them J1 Button_LED_InOut_Connector, J2 UART_Connector, Q1 NPN, Q2 NPN, U1 Pico

Commit message: Better PCB
Parts:
- removed J1: Button_LED_InOut_Connector, Connector_PinSocket_2.54mm:PinSocket_2x06_P2.54mm_Vertical
- added J3: Button_LED_InOut_Connector, Connector_PinSocket_2.54mm:PinSocket_2x06_P2.54mm_Vertical, F.Cu at (137.3, 114.0)
- moved J2 5.11 mm to (127.5, 78.5), turned to 180 degrees
- moved G*** 0.71 mm to (143.5, 121.0)
Connections:
- J2 pad 1: Net-(J2-TX) -> Net-(J2-GND)
- J2 pad 3: Net-(J2-GND) -> Net-(J2-TX)
- U1 pad 13: unconnected-(U1-GND-Pad13) -> GND
- U1 pad 28: unconnected-(U1-GND-Pad28) -> GND
- U1 pad 33: unconnected-(U1-AGND-Pad33) -> GND
Routing:
- net Net-(U1-GPIO15): track 6.08 -> 16.8 mm
- net Net-(Q1-C): track 29.5 -> 34.4 mm, vias 1 -> 0
- net GND: track 3.59 -> 0.00 mm
- net Net-(D1-A): track 18.0 -> 15.1 mm
- net +5V: track 56.9 -> 58.0 mm
- net Net-(J3-LED_OUT_+): track 14.3 -> 13.5 mm
