File: KiCad/picoswitch.kicad_sch (KiCad schematic)
At the start: 6 parts, among them J1 Button_LED_InOut_Connector, J2 UART_Connector, Q1 NPN, Q2 NPN, U1 Pico

Commit message: Better PCB
Parts:
- removed J1: Button_LED_InOut_Connector, Connector_PinSocket_2.54mm:PinSocket_2x06_P2.54mm_Vertical, symbol Library:Button_LED_InOut_Connector
- added J3: Button_LED_InOut_Connector, Connector_PinSocket_2.54mm:PinSocket_2x06_P2.54mm_Vertical, symbol Library:Button_LED_InOut_Connector
Connections:
- net GND: now also U1.13 (GND), U1.28 (GND), U1.33 (AGND), J3.1 (GND), J3.11 (POWER_SW_-), J3.4 (POWER_BTN), J3.6 (LED_OUT_-), J3.7 (LED_IN_-), J3.9 (RESET_BTN)
- net at U1.20 (GPIO15): now also J3.10 (RESET_BTN)
- net at D1.2 (A): now also J3.12 (POWER_SW_+)
- net at U1.19 (GPIO14): now also J3.3 (POWER_BTN)
- net at Q2.1 (C): now also J3.5 (LED_OUT_+)
- net at Q1.2 (B): now also J3.8 (LED_IN_+)
- net at J2.1 (GND): now also U1.8 (GND); no longer U1.6 (GPIO4)
- net at J2.3 (TX): now also U1.6 (GPIO4); no longer U1.8 (GND)
